File: schematics/Rx.kicad_sch (KiCad schematic)
At the start: 46 parts

Commit message: latest updates
Parts:
- added C1, C7: 1u, Capacitor_SMD:C_0603_1608Metric, symbol Device:C
- added J2: Conn_02x15_Counter_Clockwise, symbol Connector_Generic:Conn_02x15_Counter_Clockwise
- added U1: MCP1700T-3002E/MB, Package_TO_SOT_SMD:SOT-89-3, symbol Regulator_Linear:MCP1700-3002E_SOT89
- C10, C11: renamed from C?; value 10 pF -> 10p; footprint (none) -> Capacitor_SMD:C_0402_1005Metric; Candidate (none) -> 04025U100CAT2A
- C12, C14, C16, C17: renamed from C?; value 470 pF -> 470p; footprint (none) -> Capacitor_SMD:C_0603_1608Metric; Candidate (none) -> VJ0603D471KXXAJ
- C13: renamed from C?; value 18pF -> 18p; Candidate 0402ZK180GBS -> 0402ZK180GBSTR
- C15: renamed from C?; value 18pF -> 18p; Candidate GJM1555C1H180FB01 -> 04023U180FAT2A
- C18: renamed from C?; value 1uF -> 1u; Candidate GRM188R71A105KA61 -> CL10B105KP8NNNC
- C19, C21: renamed from C?; value 100 pF -> 100p; Candidate (none) -> C0402C101J3GAC
- C2: renamed from C?; value 100 nF -> 100n; footprint (none) -> Capacitor_SMD:C_0402_1005Metric; Candidate (none) -> CL05B104KA54PNC
- C20: renamed from C?; value 10 nF -> 10n; Candidate (none) -> 0805N103J500CT
- C22: renamed from C?; value 0.1uF -> 0.1u; footprint (none) -> Capacitor_SMD:C_0603_1608Metric; Candidate (none) -> 885382206004
- C23: renamed from C?; value 0.5 pF -> 0.5p; footprint (none) -> Capacitor_SMD:C_0402_1005Metric; Candidate (none) -> CQ0402BRNPO9BNR50
- C3: renamed from C?; footprint (none) -> Capacitor_SMD:C_0805_2012Metric; Candidate (none) -> 885382207005
- C4, C5, C6: renamed from C?; value 330 nF -> 330n; footprint (none) -> Capacitor_SMD:C_0805_2012Metric; Candidate (none) -> 885382207002
- C8: renamed from C?; value 10 nF -> 10n; footprint (none) -> Capacitor_SMD:C_0402_1005Metric; Candidate (none) -> 04025C103K4T2A
- C9: renamed from C?; value 2.2 uF -> 2.2u; footprint (none) -> Capacitor_SMD:C_0805_2012Metric; Candidate (none) -> CL21B225KAFNNNE
- L1, L2: renamed from L?; value 2.2 u -> 2.2uH; footprint (none) -> Inductor_SMD:L_0603_1608Metric; Candidate (none) -> 36501J2N2JTDG
- L3: renamed from L?; value 22 nH -> RF choke; footprint Inductor_SMD:L_0805_2012Metric -> Inductor_SMD:L_0402_1005Metric; Candidate (none) -> LQW15AN11NJ00D
- L4: renamed from L?; value 0.6nH -> RF choke; footprint (none) -> Inductor_SMD:L_0402_1005Metric; Candidate (none) -> LQW15AN11NJ00D
- R1, R2: renamed from R?; footprint (none) -> Resistor_SMD:R_0603_1608Metric; Candidate (none) -> ERA-3AEB5490V
- R10, R11: renamed from R?; footprint (none) -> Resistor_SMD:R_0603_1608Metric; Candidate (none) -> RT0603DRE074K99L
- R12, R13: renamed from R?; footprint (none) -> Resistor_SMD:R_0603_1608Metric; Candidate (none) -> AT0603DRD071KL
- R14: renamed from R?; footprint (none) -> Resistor_SMD:R_0402_1005Metric; Candidate (none) -> RC0402FR-7W100RL; now left out of the parts list
- R3, R4: renamed from R?; value 10 k -> 10k; footprint (none) -> Resistor_SMD:R_0603_1608Metric; Candidate (none) -> AT0603DRE0710KL
- R5: renamed from R?; footprint (none) -> Resistor_SMD:R_0402_1005Metric; Candidate (none) -> CRGP0402F10K; now left out of the parts list
- R6, R7: renamed from R?; footprint (none) -> Resistor_SMD:R_0603_1608Metric; Candidate (none) -> RT0603DRE07910RL
- R8, R9: renamed from R?; footprint (none) -> Resistor_SMD:R_0603_1608Metric; Candidate (none) -> RT0603DRE07130RL
- U2: renamed from U?; Candidate (none) -> LDS3985M25R
- U3: renamed from U?; COPYRIGHT Copyright C 2016 Accelerated Designs. All rights reserved -> (none); Candidate (none) -> LT6232CGN#PBF; DIGIKEY_PART_NUMBER LT6232CGN#PBFND -> (none); MANUFACTURER_PART_NUMBER LT6232CGN#PBF -> (none); VENDOR Linear Technology -> (none)
- U4: renamed from U?; Candidate (none) -> LT5552
- U5: renamed from U?; Candidate (none) -> HMC313E
- U6: renamed from U?; Candidate (none) -> SKY65404
- gave numbers to parts that had none: 2
Connections:
- net 3V0: now also C7.1, U1.3 (VO); no longer R14.2
- net GND: now also J1.2 (Ext), J3.2 (Ext), U4.12 (GND), C1.2, C7.2, J2.1 (Pin_1), J2.11 (Pin_11), J2.13 (Pin_13), J2.15 (Pin_15), J2.18 (Pin_18), J2.23 (Pin_23), J2.26 (Pin_26), J2.3 (Pin_3), J2.7 (Pin_7), U1.1 (GND)
- net IFF+: now also J2.24 (Pin_24)
- net IFF-: now also J2.25 (Pin_25)
- net MIXER_ENABLE: now also J2.29 (Pin_29)
- net RF: now reaches C19.1, U4.5 (RF)
- net 3V3 renamed +3V3
- net +3V3: now also C1.1, J2.16 (Pin_16), J2.17 (Pin_17), J2.2 (Pin_2), J2.4 (Pin_4), J2.5 (Pin_5), J2.6 (Pin_6), U1.2 (VI)
- net 5V renamed +5V
- net +5V: now also J2.10 (Pin_10), J2.12 (Pin_12), J2.8 (Pin_8), J2.9 (Pin_9)
- new net +10V: J2.14 (Pin_14)
- new net LNA_ENABLE: J2.30 (Pin_30), R14.2
- no-connect marks 0 -> 6
Other:
- note added: "3V0: 15 mA 3V3: 200 mA supply ramp time of > 1 ms 5V: 90 mA"
- moved on the sheet: C13, C15, C18, C19, C20, C21, C22, C23, J1, J3, L3, L4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
